Commit message: calib fixes

File: src/ray_trace/urdf/velma.urdf (robot description, URDF)
Before this commit: robot velma, 70 links, 69 joints
Links:
- removed link left_needle_link
- removed link right_needle_link
- link head_pan_link: geometry visual mesh filename=package://velma_description/meshes/head_tilt_simplified.STL
- link head_pan_motor: geometry visual mesh filename=package://velma_description/meshes/head_pan_simplified.STL
- link head_tilt_link: geometry visual mesh filename=package://velma_description/meshes/collision/head_top_colli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; visual mesh filename=package://velma_description/meshes/head_top_simplified.STL
- link left_arm_5_link: geometry collision mesh filename=package://lwr_defs/meshes/lwr/convex/arm_segment_last_conve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; visual mesh filename=package://lwr_defs/meshes/lwr/link_5_simplified.STL
- link left_gripper_mount_link: geometry collision mesh filename=package://velma_description/meshes/collision/gripper_mount_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; visual box size=0.02 0.02 0.005
- link right_arm_5_link: geometry collision mesh filename=package://lwr_defs/meshes/lwr/convex/arm_segment_last_conve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; visual mesh filename=package://lwr_defs/meshes/lwr/link_5_simplified.STL
- link right_gripper_mount_link: geometry collision mesh filename=package://velma_description/meshes/collision/gripper_mount_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; visual box size=0.02 0.02 0.005
- link torso_link0: geometry collision mesh filename=package://velma_description/meshes/collision/torso0_collisi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; collision sphere radius=0.24
Joints:
- removed joint left_needle_joint
- removed joint right_needle_joint

Commit message: added env yaml

File: src/ray_trace/urdf/velma.urdf (robot description, URDF)
Before this commit: robot velma, 68 links, 67 joints
Links:
- added link head_bounding_sphere, mass 0.3; collision sphere radius=0.24
Joints:
- added joint head_bounding_sphere_joint: type fixed, parent torso_base, child head_bounding_sphere, origin xyz=0 0 0.03 rpy=0 0 0
- joint torso_0_joint: limit lower=-1.57 upper=1.57 effort=100 velocity=100 -> lower=-1.57 upper=1.57 effort=100 velocity=0.523598775598
